File: OpenThermalKiCad/OpenThermal/OpenThermal.kicad_pcb (KiCad board)
At the start: 2 copper layers, 86.4 x 81.3 mm, 7 parts, among them U1 MLX90621ESF-BAB-000-SP

Commit message: Updated camera module
Parts:
- PWR_IN1: footprint Connector_PinSocket_2.54mm:PinSocket_1x04_P2.54mm_Vertical -> Connector_PinSocket_2.54mm:PinSocket_1x03_P2.54mm_Vertical
- moved U1 70.3 mm to (175.3, 101.6), turned to -90 degrees
- moved C1 58.4 mm to (167.6, 102.8), turned to 90 degrees
Connections:
- PWR_IN1 pad 2: BatteryLatch -> GND1
- PWR_IN1 pad 3: GND1 -> +5V
- PWR_OUT1 pad 4: +3.3V -> +5V
- esp1 pad 22: SPI_MOSI -> SPI_CLOCK
- esp1 pad 25: SPI_CLOCK -> SPI_MOSI
- esp1 pad 27: MLX_SDA -> SPI_CS1
- esp1 pad 28: MLX_SCL -> SPI_CS2
- esp1 pad 29: BatteryLatch -> unconnected-(esp1-G5-Pad29)
- esp1 pad 30: SPI_CS1 -> MLX_SDA
- esp1 pad 31: SPI_CS2 -> MLX_SCL
Routing:
- net +3.3V: track 55.6 -> 142.9 mm
- net +5V: track 13.3 -> 82.5 mm
- net BatteryLatch: track 38.3 -> 0.00 mm
- net MLX_SCL: track 49.9 -> 37.9 mm
- net MLX_SDA: track 49.9 -> 37.9 mm
- net SPI_CS1: track 24.1 -> 31.8 mm
- net BatteryLevel: track 22.0 -> 25.7 mm
- net SPI_CS2: track 30.2 -> 31.9 mm
- net GND1: track 51.4 -> 50.4 mm
Other:
- board size 86.4 x 81.3 mm -> 73.7 x 81.3 mm
- board text added: "5V"
- board text removed: "LATCH"
