File: OpenThermalKiCad/OpenThermal/OpenThermal.kicad_sch (KiCad schematic)
At the start: 7 parts, among them U1 MLX90621ESF-BAB-000-SP

Commit message: Updated camera module
Parts:
- PWR_IN1: footprint Connector_PinSocket_2.54mm:PinSocket_1x04_P2.54mm_Vertical -> Connector_PinSocket_2.54mm:PinSocket_1x03_P2.54mm_Vertical; symbol Connector_Generic:Conn_01x04 -> Connector_Generic:Conn_01x03
Connections:
- net +3.3V: no longer PWR_OUT1.4 (Pin_4)
- net +5V: now also PWR_IN1.3 (Pin_3), PWR_OUT1.4 (Pin_4); no longer PWR_IN1.4 (Pin_4)
- net GND1: now also PWR_IN1.2 (Pin_2); no longer PWR_IN1.3 (Pin_3)
- net MLX_SCL: now also esp1.31 (G16); no longer esp1.28 (G18)
- net MLX_SDA: now also esp1.30 (G17); no longer esp1.27 (G19)
- net SPI_CLOCK: now also esp1.22 (G22); no longer esp1.25 (G21)
- net SPI_CS1: now also esp1.27 (G19); no longer esp1.30 (G17)
- net SPI_CS2: now also esp1.28 (G18); no longer esp1.31 (G16)
- net SPI_MOSI: now also esp1.25 (G21); no longer esp1.22 (G22)
- net BatteryLatch: no longer names the net of esp1.29 (G5)
- net BatteryLatch: no longer PWR_IN1.2 (Pin_2)
Other:
- moved on the sheet: PWR_OUT1, SPI1, SPI2
