File: OpenThermalKiCad/OpenThermalMainboard/OpenThermalMainboard.kicad_pcb (KiCad board)
At the start: 2 copper layers, 78.7 x 81.3 mm, 7 parts, among them U1 MLX90621ESF-BAB-000-SP

Commit message: Updated wiring and placement
Parts:
- moved esp1 2.54 mm to (48.3, 58.4)
Routing:
- net SPI_CLOCK: track 36.9 -> 23.9 mm
- net SPI_MISO: track 36.9 -> 23.9 mm
- net SPI_MOSI: track 36.9 -> 26.0 mm
- net SPI_CS1: track 31.8 -> 22.0 mm
- net +3.3V: track 137.0 -> 141.3 mm
- net +5V: track 79.5 -> 83.6 mm
- net MLX_SCL: track 37.9 -> 33.9 mm
- net MLX_SDA: track 37.9 -> 34.1 mm
- net SPI_CS2: track 31.9 -> 28.1 mm
- net GND1: track 47.4 -> 44.8 mm
- net BatteryLevel: track 25.0 -> 23.2 mm

Commit message: Updated wiring + components
Parts:
- moved SPI2 13.7 mm to (78.7, 25.4), turned to 90 degrees
- moved SPI1 7.62 mm to (78.7, 30.5), turned to 90 degrees
Routing:
- net SPI_CS2: track 28.1 -> 50.1 mm
- net SPI_CS1: track 22.0 -> 40.4 mm
- net SPI_MOSI: track 26.0 -> 39.3 mm
- net SPI_CLOCK: track 23.9 -> 32.1 mm
- net SPI_MISO: track 23.9 -> 27.1 mm
- net MLX_SCL: track 33.9 -> 32.2 mm
- net MLX_SDA: track 34.1 -> 33.0 mm
Other:
- board size 78.7 x 81.3 mm -> 88.9 x 83.8 mm

Commit message: Updated main
Routing:
- net SPI_CS2: track 50.1 -> 51.6 mm
Changed lines of the file:
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@@
   (segment (start 81.28 30.48) (end 81.28 33.02) (width 0.3) (layer "F.Cu") (net 32))
   (segment (start 81.28 33.02) (end 71.12 43.18) (width 0.3) (layer "F.Cu") (net 32))
-  (segment (start 88.9 38.1) (end 68.58 58.42) (width 0.3) (layer "F.Cu") (net 33))
+  (segment (start 71.12 58.42) (end 60.96 58.42) (width 0.3) (layer "F.Cu") (net 33))
+  (segment (start 88.9 27.94) (end 88.9 40.64) (width 0.3) (layer "F.Cu") (net 33))
   (segment (start 86.36 25.4) (end 88.9 27.94) (width 0.3) (layer "F.Cu") (net 33))
-  (segment (start 68.58 58.42) (end 60.96 58.42) (width 0.3) (layer "F.Cu") (net 33))
-  (segment (start 88.9 27.94) (end 88.9 38.1) (width 0.3) (layer "F.Cu") (net 33))
+  (segment (start 88.9 40.64) (end 71.12 58.42) (width 0.3) (layer "F.Cu") (net 33))
   (segment (start 86.36 38.1) (end 68.58 55.88) (width 0.3) (layer "F.Cu") (net 34))
   (segment (start 86.36 30.48) (end 86.36 38.1) (width 0.3) (layer "F.Cu") (net 34))
